File: board/board.kicad_pcb (KiCad board)
At the start: 2 copper layers, 21 x 13 mm, 1 part

Commit message: imported legacy
Parts:
- removed LOGO1: Logo_Open_Hardware_Small, Symbol:OSHW-Symbol_6.7x6mm_SilkScreen
- added C1: 100nF, Capacitor_SMD:C_0603_1608Metric, F.Cu at (154.8, 99.1)
- added J1: 021_single_IO_UNIO, on_edge:on_edge_2x05_device, F.Cu at (141.5, 99.0)
- added U1: 11AA02E48, Package_TO_SOT_SMD:SOT-23, F.Cu at (151.0, 98.8)
Routing:
- net GND: track 0.00 -> 13.5 mm
- net /mac/3.3V: track 0.00 -> 11.5 mm, vias 0 -> 1
- net /mac/IO: track 0.00 -> 6.56 mm
Other:
- board size 21 x 13 mm -> 22 x 13 mm
- copper layers 2 -> 4
- rule pad_to_mask_clearance: 0 -> 0.051
- board text added: "osf.b096.v0.1"
