File: board/board.kicad_sch (KiCad schematic)
At the start: 1 part

Commit message: imported legacy
Parts:
- removed LOGO1: Logo_Open_Hardware_Small, Symbol:OSHW-Symbol_6.7x6mm_SilkScreen, symbol Graphic:Logo_Open_Hardware_Small
- added C1: 100nF, Capacitor_SMD:C_0603_1608Metric, symbol Device:C_Small
- added J1: 021_single_IO_UNIO, on_edge:on_edge_2x05_device, symbol put_on_edge:021_single_IO_UNIO
Connections:
- new net GND: C1.2, J1.1 (GND)
- new net mac/3.3V: C1.1, J1.9 (3.3V)
- new net mac/IO: J1.2 (SCIO)
- no-connect marks 0 -> 1
Other:
- removed sheet implementation
- added sheet mac (mac.kicad_sch)
- note removed: "Input connectors go here"
- note removed: "Output connectors go here"
Changed lines of the file:
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@@
 (kicad_sch (version 20211123) (generator eeschema)
   (paper "A4")
-  (text "Output connectors go here" (at 224.79 88.9 0)
-    (effects (font (size 1.27 1.27)) (justify left bottom))
+  (junction (at 73.66 97.79) (diameter 0) (color 0 0 0 0)
   )
-  (text "Input connectors go here" (at 49.53 88.9 0)
-    (effects (font (size 1.27 1.27)) (justify left bottom))
+  (no_connect (at 58.42 100.33))
+  (wire (pts (xy 58.42 87.63) (xy 95.25 87.63))
+    (stroke (width 0) (type default) (color 0 0 0 0))
   )
-  (symbol (lib_id "Graphic:Logo_Open_Hardware_Small") (at 273.05 157.48 0) (unit 1)
+  (wire (pts (xy 92.71 104.14) (xy 95.25 104.14))
+    (stroke (width 0) (type default) (color 0 0 0 0))
+  )
+  (wire (pts (xy 92.71 109.22) (xy 92.71 104.14))
+    (stroke (width 0) (type default) (color 0 0 0 0))
+  )
+  (wire (pts (xy 73.66 97.79) (xy 95.25 97.79))
+    (stroke (width 0) (type default) (color 0 0 0 0))
+  )
+  (wire (pts (xy 58.42 97.79) (xy 73.66 97.79))
+    (stroke (width 0) (type default) (color 0 0 0 0))
+  )
+  (wire (pts (xy 73.66 102.87) (xy 73.66 97.79))
+    (stroke (width 0) (type default) (color 0 0 0 0))
+  )
+  (symbol (lib_id "power:GND") (at 48.26 109.22 0) (unit 1)
     (in_bom yes) (on_board yes) (fields_autoplaced)
-    (property "Reference" "LOGO1" (id 0) (at 273.05 150.495 0)
+    (property "Reference" "#PWR0101" (id 0) (at 48.26 115.57 0)
       (effects (font (size 1.27 1.27)) hide)
     )
-    (property "Value" "Logo_Open_Hardware_Small" (id 1) (at 273.05 163.195 0)
+    (property "Value" "GND" (id 1) (at 48.26 114.3 0))
+    (property "Footprint" "" (id 2) (at 48.26 109.22 0)
       (effects (font (size 1.27 1.27)) hide)
     )
-    (property "Footprint" "Symbol:OSHW-Symbol_6.7x6mm_SilkScreen" (id 2) (at 273.05 157.48 0)
+    (property "Datasheet" "" (id 3) (at 48.26 109.22 0)
       (effects (font (size 1.27 1.27)) hide)
     )
-    (property "Datasheet" "~" (id 3) (at 273.05 157.48 0)
+    (pin "1")
+  )
+  (symbol (lib_id "power:GND") (at 73.66 107.95 0) (unit 1)
+    (in_bom yes) (on_board yes) (fields_autoplaced)
+    (property "Reference" "#PWR0103" (id 0) (at 73.66 114.3 0)
       (effects (font (size 1.27 1.27)) hide)
     )
+    (property "Value" "GND" (id 1) (at 73.66 113.03 0))
+    (property "Footprint" "" (id 2) (at 73.66 107.95 0)
+      (effects (font (size 1.27 1.27)) hide)
+    )
+    (property "Datasheet" "" (id 3) (at 73.66 107.95 0)
+      (effects (font (size 1.27 1.27)) hide)
+    )
+    (pin "1")
   )
-  (sheet (at 114.3 72.39) (size 60.96 62.23) (fields_autoplaced)
+  (symbol (lib_id "put_on_edge:021_single_IO_UNIO") (at 46.99 95.25 0) (mirror y) (unit 1)
+    (in_bom yes) (on_board yes) (fields_autoplaced)
+    (property "Reference" "J1" (id 0) (at 47.625 77.47 0))
+    (property "Value" "021_single_IO_UNIO" (id 1) (at 47.625 80.01 0))
+    (property "Footprint" "on_edge:on_edge_2x05_device" (id 2) (at 39.37 78.74 0)
+      (effects (font (size 1.27 1.27)) hide)
+    )
+    (property "Datasheet" "" (id 3) (at 39.37 78.74 0)
+      (effects (font (size 1.27 1.27)) hide)
+    )
+    (pin "1")
+    (pin "10")
+    (pin "2")
+    (pin "9")
+  )
+  (symbol (lib_id "Device:C_Small") (at 73.66 105.41 0) (unit 1)
+    (in_bom yes) (on_board yes) (fields_autoplaced)
+    (property "Reference" "C1" (id 0) (at 76.2 104.1462 0)
+      (effects (font (size 1.27 1.27)) (justify left))
+    )
+    (property "Value" "100nF" (id 1) (at 76.2 106.6862 0)
+      (effects (font (size 1.27 1.27)) (justify left))
+    )
+    (property "Footprint" "Capacitor_SMD:C_0603_1608Metric" (id 2) (at 73.66 105.41 0)
+      (effects (font (size 1.27 1.27)) hide)
+    )
+    (property "Datasheet" "~" (id 3) (at 73.66 105.41 0)
+      (effects (font (size 1.27 1.27)) hide)
+    )
+    (pin "1")
+    (pin "2")
+  )
+  (symbol (lib_id "power:GND") (at 92.71 109.22 0) (unit 1)
+    (in_bom yes) (on_board yes) (fields_autoplaced)
+    (property "Reference" "#PWR0102" (id 0) (at 92.71 115.57 0)
+      (effects (font (size 1.27 1.27)) hide)
+    )
+    (property "Value" "GND" (id 1) (at 92.71 114.3 0))
+    (property "Footprint" "" (id 2) (at 92.71 109.22 0)
+      (effects (font (size 1.27 1.27)) hide)
+    )
+    (property "Datasheet" "" (id 3) (at 92.71 109.22 0)
+      (effects (font (size 1.27 1.27)) hide)
+    )
+    (pin "1")
+  )
+  (sheet (at 95.25 82.55) (size 20.32 24.13) (fields_autoplaced)
     (stroke (width 0.1524) (type solid) (color 0 0 0 0))
     (fill (color 0 0 0 0.0000))
-    (property "Sheet name" "implementation" (id 0) (at 114.3 71.6784 0)
+    (property "Sheet name" "mac" (id 0) (at 95.25 81.8384 0)
       (effects (font (size 1.27 1.27)) (justify left bottom))
     )
-    (property "Sheet file" "implementation.kicad_sch" (id 1) (at 114.3 135.2046 0)
+    (property "Sheet file" "mac.kicad_sch" (id 1) (at 95.25 107.2646 0)
       (effects (font (size 1.27 1.27)) (justify left top))
+    )
+    (pin "GND" input (at 95.25 104.14 180)
+      (effects (font (size 1.27 1.27)) (justify left))
+    )
+    (pin "3.3V" input (at 95.25 97.79 180)
+      (effects (font (size 1.27 1.27)) (justify left))
+    )
+    (pin "IO" input (at 95.25 87.63 180)
+      (effects (font (size 1.27 1.27)) (justify left))
     )
   )
   (sheet_instances
     (path "/" (page "1"))
-    (path "/767ce4c6-0e55-4543-92f0-34cb8237a544" (page "2"))
+    (path "/e63fd82c-ac1a-4b5a-b264-e2fd55c97b9a" (page "2"))
   )
   (symbol_instances
-    (path "/b72b6f4a-7489-40f2-bb90-d75ae01aa368"
-      (reference "LOGO1") (unit 1) (value "Logo_Open_Hardware_Small") (footprint "Symbol:OSHW-Symbol_6.7x6mm_SilkScreen")
+    (path "/0360b572-41f0-4961-997b-aba63f8c11ae"
+      (reference "#PWR0101") (unit 1) (value "GND") (footprint "")
+    )
+    (path "/fa2197e2-1e78-4a6c-99e8-4d65757a2793"
+      (reference "#PWR0102") (unit 1) (value "GND") (footprint "")
+    )
+    (path "/0549e634-4477-4836-a1eb-e4641251bafe"
+      (reference "#PWR0103") (unit 1) (value "GND") (footprint "")
+    )
+    (path "/8ee79578-7e3a-49b2-b893-a8b807ce503b"
+      (reference "C1") (unit 1) (value "100nF") (footprint "Capacitor_SMD:C_0603_1608Metric")
+    )
+    (path "/41ad0fc7-b163-4156-ae80-0e575916d9c7"
+      (reference "J1") (unit 1) (value "021_single_IO_UNIO") (footprint "on_edge:on_edge_2x05_device")
+    )
+    (path "/e63fd82c-ac1a-4b5a-b264-e2fd55c97b9a/cb2ba9a4-f213-49d9-ba66-a6034b621a6f"
+      (reference "U1") (unit 1) (value "11AA02E48") (footprint "Package_TO_SOT_SMD:SOT-23")
     )
   )
